Commit message: Fix Suivi Cap et ajout mesh

File: ros2_ws/src/benoit_pairob/src/description/benoit_pairob_description.urdf (robot description, URDF)
Before this commit: robot benoit_pairob, 9 links, 8 joints
Links:
- removed link front_caster
- removed link front_left_link
- removed link front_link
- removed link front_right_link
- added link left_caster; collision sphere radius=${(wheel_radius+wheel_zoff-(base_height/2))}; visual sphere radius=${(wheel_radius+wheel_zoff-(base_height/2))}
- added link right_caster; collision sphere radius=${(wheel_radius+wheel_zoff-(base_height/2))}; visual sphere radius=${(wheel_radius+wheel_zoff-(base_height/2))}
- link base_link: geometry collision box size=${base_length} ${base_width} ${base_height}; visual mesh filename=file://$(find benoit_pairob)/src/description/meshes/Chassis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
Joints:
- removed joint caster_joint
- removed joint front_joint
- removed joint front_left_joint
- removed joint front_right_joint
- added joint left_caster_joint: type fixed, parent base_link, child left_caster, origin xyz=${caster_xoff} 0.0 ${-(base_height/2)} rpy=0 0 0
- added joint right_caster_joint: type fixed, parent base_link, child right_caster, origin xyz=${caster_xoff} 0.0 ${-(base_height/2)} rpy=0 0 0

Commit message: Fix collision

File: ros2_ws/src/benoit_pairob/src/description/benoit_pairob_description.urdf (robot description, URDF)
Before this commit: robot benoit_pairob, 7 links, 6 joints
Links:
- link base_link: geometry collision mesh filename=file://$(find benoit_pairob)/src/description/meshes/Chassis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; visual mesh filename=file://$(find benoit_pairob)/src/description/meshes/Chassis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
